File: prototype_board/TCS3414_v0.brd (EAGLE design)
At the start: 43.2 x 22.9 mm, 6 parts, among them U1 TCS3414FNFN

Commit message: Changed resistor values
2.5k to 10k and 1.3k to 4.7k resistor changes
Parts:
- R1: value 2k5 -> 10k
- R2, R3: value 1k3 -> 4k7
Changed lines of the file:
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@@
 <?xml version="1.0" encoding="utf-8"?>
 <!DOCTYPE eagle SYSTEM "eagle.dtd">
-<eagle version="7.4.0">
+<eagle version="6.6.0">
 <drawing>
 <settings>
@@
 <pass name="Default">
 <param name="RoutingGrid" value="50mil"/>
-<param name="AutoGrid" value="1"/>
-<param name="Efforts" value="0"/>
-<param name="TopRouterVariant" value="1"/>
 <param name="tpViaShape" value="round"/>
-<param name="PrefDir.1" value="a"/>
+<param name="PrefDir.1" value="|"/>
 <param name="PrefDir.2" value="0"/>
 <param name="PrefDir.3" value="0"/>
@@
 <param name="PrefDir.14" value="0"/>
 <param name="PrefDir.15" value="0"/>
-<param name="PrefDir.16" value="a"/>
+<param name="PrefDir.16" value="-"/>
 <param name="cfVia" value="8"/>
 <param name="cfNonPref" value="5"/>
@@
 <elements>
 <element name="C1" library="resistor" package="C0603" value="0.1uF" x="38.1" y="25.4" rot="R180"/>
-<element name="R1" library="rcl" package="R0603" value="2k5" x="30.48" y="25.4"/>
-<element name="R2" library="rcl" package="R0603" value="1k3" x="29.21" y="31.75"/>
-<element name="R3" library="rcl" package="R0603" value="1k3" x="43.18" y="31.75" rot="R270"/>
+<element name="R1" library="rcl" package="R0603" value="10k" x="30.48" y="25.4"/>
+<element name="R2" library="rcl" package="R0603" value="4k7" x="29.21" y="31.75"/>
+<element name="R3" library="rcl" package="R0603" value="4k7" x="43.18" y="31.75" rot="R270"/>
 <element name="U$1" library="mcu-accessories" package="TEENSY_3.1_BASIC" value="TEENSY_3.1_BASIC" x="34.29" y="29.21" rot="MR90"/>
 <element name="U1" library="TCS3414FN" package="TCS3414FN" value="TCS3414FNFN" x="35.56" y="30.48" rot="R270"/>
