File: wavemeter/sensorBoard_1.0.sch (EAGLE design)
At the start: 4 parts, among them J1 MJACK8P8CVERT, U1 TCS3414FN, U2 ADS1118RUG

Commit message: Clean up and organization of folders
Also fixed crossed MOSI/MISO wires on the teensyBoard eagle files
Connections:
- net N$7: now also J1.MISO; no longer J1.DOUT
- net N$8: now also J1.MOSI; no longer J1.DIN
Changed lines of the file:
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@@
 <pinref part="U2" gate="G$1" pin="DOUT"/>
 <wire x1="33.02" y1="24.638" x2="121.92" y2="24.638" width="0.1524" layer="91"/>
-<pinref part="J1" gate="G$1" pin="DOUT"/>
+<pinref part="J1" gate="G$1" pin="MISO"/>
 <wire x1="38.1" y1="43.18" x2="33.02" y2="43.18" width="0.1524" layer="91"/>
 <wire x1="33.02" y1="43.18" x2="33.02" y2="25.146" width="0.1524" layer="91"/>
@@
 <pinref part="U2" gate="G$1" pin="DIN"/>
 <wire x1="22.86" y1="22.86" x2="22.86" y2="53.34" width="0.1524" layer="91"/>
-<pinref part="J1" gate="G$1" pin="DIN"/>
+<pinref part="J1" gate="G$1" pin="MOSI"/>
 <wire x1="22.86" y1="53.34" x2="38.1" y2="53.34" width="0.1524" layer="91"/>
 </segment>
